File: 2070-S-100-bus-analyzer.kicad_pcb (KiCad board)
At the start: 2 copper layers, 254 x 134.6 mm, 3 parts, among them J1 S100

Commit message: Re-start project from new KiCad9 S-100 template
Parts:
- H1, H2: value Ejector -> MountingHole; footprint jb-footprint:MountingHole_2.7mm_M2.5 -> MountingHole:MountingHole_2.5mm
- J1: value S100 -> ~; footprint jb-footprint:S100_MALE -> S100-footprints:S100-Edge-Connector
- moved J1 74.7 mm to (138.4, 158.8)
- moved H2 6.35 mm to (266.7, 31.8)
- moved H1 6.35 mm to (25.4, 31.8)
Connections:
- J1 pad 1: Net-(J1-Pad1) -> unconnected-(J1-+8-Pad1)
- J1 pad 10: Net-(J1-Pad10) -> unconnected-(J1-~{VI6}-Pad10)
- J1 pad 100: Net-(J1-Pad100) -> unconnected-(J1-GND-Pad100)
- J1 pad 11: Net-(J1-Pad11) -> unconnected-(J1-~{VI7}-Pad11)
- J1 pad 12: Net-(J1-Pad12) -> unconnected-(J1-~{NMI}-Pad12)
- J1 pad 13: Net-(J1-Pad13) -> unconnected-(J1-~{PWRFAIL}-Pad13)
- J1 pad 14: Net-(J1-Pad14) -> unconnected-(J1-~{DMA3}-Pad14)
- J1 pad 15: Net-(J1-Pad15) -> unconnected-(J1-A18-Pad15)
- J1 pad 16: Net-(J1-Pad16) -> unconnected-(J1-A16-Pad16)
- J1 pad 17: Net-(J1-Pad17) -> unconnected-(J1-A17-Pad17)
- J1 pad 18: Net-(J1-Pad18) -> unconnected-(J1-~{SDSB}-Pad18)
- J1 pad 19: Net-(J1-Pad19) -> unconnected-(J1-~{CDSB}-Pad19)
- J1 pad 2: Net-(J1-Pad2) -> unconnected-(J1-+16-Pad2)
- J1 pad 20: Net-(J1-Pad20) -> unconnected-(J1-GND-Pad20)
- J1 pad 21: Net-(J1-Pad21) -> unconnected-(J1-NDEF-Pad21)
- J1 pad 22: Net-(J1-Pad22) -> unconnected-(J1-~{ADBB}-Pad22)
- J1 pad 23: Net-(J1-Pad23) -> unconnected-(J1-~{DODSB}-Pad23)
- J1 pad 24: Net-(J1-Pad24) -> unconnected-(J1-PHI-Pad24)
- J1 pad 25: Net-(J1-Pad25) -> unconnected-(J1-~{pSTVAL}-Pad25)
- J1 pad 26: Net-(J1-Pad26) -> unconnected-(J1-pHLDA-Pad26)
- J1 pad 27: Net-(J1-Pad27) -> unconnected-(J1-RFU-Pad27)
- J1 pad 28: Net-(J1-Pad28) -> unconnected-(J1-RFU-Pad28)
- J1 pad 29: Net-(J1-Pad29) -> unconnected-(J1-A5-Pad29)
- J1 pad 3: Net-(J1-Pad3) -> unconnected-(J1-XRDY-Pad3)
- J1 pad 30: Net-(J1-Pad30) -> unconnected-(J1-A4-Pad30)
- J1 pad 31: Net-(J1-Pad31) -> unconnected-(J1-A3-Pad31)
- J1 pad 32: Net-(J1-Pad32) -> unconnected-(J1-A15-Pad32)
- J1 pad 33: Net-(J1-Pad33) -> unconnected-(J1-A12-Pad33)
- J1 pad 34: Net-(J1-Pad34) -> unconnected-(J1-A9-Pad34)
- J1 pad 35: Net-(J1-Pad35) -> unconnected-(J1-DO1-Pad35)
- J1 pad 36: Net-(J1-Pad36) -> unconnected-(J1-DO0-Pad36)
- J1 pad 37: Net-(J1-Pad37) -> unconnected-(J1-A10-Pad37)
- J1 pad 38: Net-(J1-Pad38) -> unconnected-(J1-DO4-Pad38)
- J1 pad 39: Net-(J1-Pad39) -> unconnected-(J1-DO5-Pad39)
- J1 pad 4: Net-(J1-Pad4) -> unconnected-(J1-~{VI0}-Pad4)
- J1 pad 40: Net-(J1-Pad40) -> unconnected-(J1-DO6-Pad40)
- J1 pad 41: Net-(J1-Pad41) -> unconnected-(J1-DI2-Pad41)
- J1 pad 42: Net-(J1-Pad42) -> unconnected-(J1-DI3-Pad42)
- J1 pad 43: Net-(J1-Pad43) -> unconnected-(J1-DI7-Pad43)
- J1 pad 44: Net-(J1-Pad44) -> unconnected-(J1-sM1-Pad44)
- J1 pad 45: Net-(J1-Pad45) -> unconnected-(J1-sOUT-Pad45)
- J1 pad 46: Net-(J1-Pad46) -> unconnected-(J1-sINP-Pad46)
- J1 pad 47: Net-(J1-Pad47) -> unconnected-(J1-sMEMR-Pad47)
- J1 pad 48: Net-(J1-Pad48) -> unconnected-(J1-sHLTA-Pad48)
- J1 pad 49: Net-(J1-Pad49) -> unconnected-(J1-CLOCK-Pad49)
- J1 pad 5: Net-(J1-Pad5) -> unconnected-(J1-~{VI1}-Pad5)
- J1 pad 50: Net-(J1-Pad50) -> unconnected-(J1-GND-Pad50)
- J1 pad 51: Net-(J1-Pad51) -> unconnected-(J1-+8-Pad51)
- J1 pad 52: Net-(J1-Pad52) -> unconnected-(J1--16-Pad52)
- J1 pad 53: Net-(J1-Pad53) -> unconnected-(J1-GND-Pad53)
- J1 pad 54: Net-(J1-Pad54) -> unconnected-(J1-~{SLV_CLR}-Pad54)
- J1 pad 55: Net-(J1-Pad55) -> unconnected-(J1-~{DMA0}-Pad55)
- J1 pad 56: Net-(J1-Pad56) -> unconnected-(J1-~{DMA1}-Pad56)
- J1 pad 57: Net-(J1-Pad57) -> unconnected-(J1-~{DMA2}-Pad57)
- J1 pad 58: Net-(J1-Pad58) -> unconnected-(J1-~{sXTRQ}-Pad58)
- J1 pad 59: Net-(J1-Pad59) -> unconnected-(J1-A19-Pad59)
- J1 pad 6: Net-(J1-Pad6) -> unconnected-(J1-~{VI2}-Pad6)
- J1 pad 60: Net-(J1-Pad60) -> unconnected-(J1-~{SIXTN}-Pad60)
- J1 pad 61: Net-(J1-Pad61) -> unconnected-(J1-A20-Pad61)
- J1 pad 62: Net-(J1-Pad62) -> unconnected-(J1-A21-Pad62)
- J1 pad 63: Net-(J1-Pad63) -> unconnected-(J1-A22-Pad63)
- J1 pad 64: Net-(J1-Pad64) -> unconnected-(J1-A23-Pad64)
- J1 pad 65: Net-(J1-Pad65) -> unconnected-(J1-NDEF-Pad65)
- J1 pad 66: Net-(J1-Pad66) -> unconnected-(J1-NDEF-Pad66)
- J1 pad 67: Net-(J1-Pad67) -> unconnected-(J1-~{PHANTOM}-Pad67)
- J1 pad 68: Net-(J1-Pad68) -> unconnected-(J1-MWRT-Pad68)
- J1 pad 69: Net-(J1-Pad69) -> unconnected-(J1-RFU-Pad69)
- J1 pad 7: Net-(J1-Pad7) -> unconnected-(J1-~{VI3}-Pad7)
- J1 pad 70: Net-(J1-Pad70) -> unconnected-(J1-GND-Pad70)
- J1 pad 71: Net-(J1-Pad71) -> unconnected-(J1-RFU-Pad71)
- J1 pad 72: Net-(J1-Pad72) -> unconnected-(J1-RDY-Pad72)
- J1 pad 73: Net-(J1-Pad73) -> unconnected-(J1-~{INT}-Pad73)
- J1 pad 74: Net-(J1-Pad74) -> unconnected-(J1-~{HOLD}-Pad74)
- J1 pad 75: Net-(J1-Pad75) -> unconnected-(J1-~{RESET}-Pad75)
- J1 pad 76: Net-(J1-Pad76) -> unconnected-(J1-pSYNC-Pad76)
- J1 pad 77: Net-(J1-Pad77) -> unconnected-(J1-~{pWR}-Pad77)
- J1 pad 78: Net-(J1-Pad78) -> unconnected-(J1-pDBIN-Pad78)
- J1 pad 79: Net-(J1-Pad79) -> unconnected-(J1-A0-Pad79)
- J1 pad 8: Net-(J1-Pad8) -> unconnected-(J1-~{VI4}-Pad8)
- J1 pad 80: Net-(J1-Pad80) -> unconnected-(J1-A1-Pad80)
- J1 pad 81: Net-(J1-Pad81) -> unconnected-(J1-A2-Pad81)
- J1 pad 82: Net-(J1-Pad82) -> unconnected-(J1-A6-Pad82)
- J1 pad 83: Net-(J1-Pad83) -> unconnected-(J1-A7-Pad83)
- J1 pad 84: Net-(J1-Pad84) -> unconnected-(J1-A8-Pad84)
- J1 pad 85: Net-(J1-Pad85) -> unconnected-(J1-A13-Pad85)
- J1 pad 86: Net-(J1-Pad86) -> unconnected-(J1-A14-Pad86)
- J1 pad 87: Net-(J1-Pad87) -> unconnected-(J1-A11-Pad87)
- J1 pad 88: Net-(J1-Pad88) -> unconnected-(J1-DO2-Pad88)
- J1 pad 89: Net-(J1-Pad89) -> unconnected-(J1-DO3-Pad89)
- J1 pad 9: Net-(J1-Pad9) -> unconnected-(J1-~{VI5}-Pad9)
- J1 pad 90: Net-(J1-Pad90) -> unconnected-(J1-DO7-Pad90)
- J1 pad 91: Net-(J1-Pad91) -> unconnected-(J1-DI4-Pad91)
- J1 pad 92: Net-(J1-Pad92) -> unconnected-(J1-DI5-Pad92)
- J1 pad 93: Net-(J1-Pad93) -> unconnected-(J1-DI6-Pad93)
- J1 pad 94: Net-(J1-Pad94) -> unconnected-(J1-DI1-Pad94)
- J1 pad 95: Net-(J1-Pad95) -> unconnected-(J1-DI0-Pad95)
- J1 pad 96: Net-(J1-Pad96) -> unconnected-(J1-sINTA-Pad96)
- J1 pad 97: Net-(J1-Pad97) -> unconnected-(J1-~{sWO}-Pad97)
- J1 pad 98: Net-(J1-Pad98) -> unconnected-(J1-~{ERROR}-Pad98)
- J1 pad 99: Net-(J1-Pad99) -> unconnected-(J1-~{POC}-Pad99)
Other:
- board size 254 x 134.6 mm -> 254 x 137.8 mm
- rule pad_to_mask_clearance: 0.051 -> 0
- board text removed: "-"

Commit message: Checkpoint
Parts:
- added A1: RaspberryPi_Pico, Module:RaspberryPi_Pico_Common_Unspecified, F.Cu at (73.1, 52.6)
- added A2: RaspberryPi_Pico, Module:RaspberryPi_Pico_Common_Unspecified, F.Cu at (106.7, 53.1)
- added A3: RaspberryPi_Pico, Module:RaspberryPi_Pico_Common_Unspecified, F.Cu at (139.7, 53.3)
- added A4: RaspberryPi_Pico, Module:RaspberryPi_Pico_Common_Unspecified, F.Cu at (174.0, 53.3)
- added A5: RaspberryPi_Pico, Module:RaspberryPi_Pico_Common_Unspecified, F.Cu at (225.0, 52.6)
- added D1: LED_Filled, LED_SMD:LED_0805_2012Metric_Pad1.15x1.40mm_HandSolder, F.Cu at (53.3, 31.5)
- added D2: LED_Filled, LED_SMD:LED_0805_2012Metric_Pad1.15x1.40mm_HandSolder, F.Cu at (50.8, 31.5)
- added D3: LED_Filled, LED_SMD:LED_0805_2012Metric_Pad1.15x1.40mm_HandSolder, F.Cu at (48.3, 31.5)
- added J10: Conn_02x13_Odd_Even, Connector_PinHeader_2.54mm:PinHeader_2x13_P2.54mm_Vertical, F.Cu at (229.3, 127.5)
- added J11: Conn_02x13_Odd_Even, Connector_PinHeader_2.54mm:PinHeader_2x13_P2.54mm_Vertical, F.Cu at (229.3, 120.4)
- added J2: Conn_02x13_Odd_Even, Connector_PinHeader_2.54mm:PinHeader_2x13_P2.54mm_Vertical, F.Cu at (70.1, 140.7)
- added J3: Conn_02x13_Odd_Even, Connector_PinHeader_2.54mm:PinHeader_2x13_P2.54mm_Vertical, F.Cu at (108.2, 140.7)
- added J4: Conn_02x13_Odd_Even, Connector_PinHeader_2.54mm:PinHeader_2x13_P2.54mm_Vertical, F.Cu at (145.8, 140.7)
- added J5: Conn_02x13_Odd_Even, Connector_PinHeader_2.54mm:PinHeader_2x13_P2.54mm_Vertical, F.Cu at (183.4, 140.7)
- added J6: Conn_02x13_Odd_Even, Connector_PinHeader_2.54mm:PinHeader_2x13_P2.54mm_Vertical, F.Cu at (70.1, 134.1)
- added J7: Conn_02x13_Odd_Even, Connector_PinHeader_2.54mm:PinHeader_2x13_P2.54mm_Vertical, F.Cu at (108.2, 134.1)
- added J8: Conn_02x13_Odd_Even, Connector_PinHeader_2.54mm:PinHeader_2x13_P2.54mm_Vertical, F.Cu at (145.8, 134.1)
- added J9: Conn_02x13_Odd_Even, Connector_PinHeader_2.54mm:PinHeader_2x13_P2.54mm_Vertical, F.Cu at (183.4, 134.1)
- added REF**: OSHW-Logo_11.4x12mm_SilkScreen, Symbol:OSHW-Logo_11.4x12mm_SilkScreen, F.Cu at (259.5, 144.0)
- added U1: 74LVCH245APW,118, Package_SO:TSSOP-20_4.4x6.5mm_P0.65mm, F.Cu at (73.7, 111.8)
- added U10: 74LVCH245APW,118, Package_SO:TSSOP-20_4.4x6.5mm_P0.65mm, F.Cu at (187.3, 111.4)
- added U11: 74LVCH245APW,118, Package_SO:TSSOP-20_4.4x6.5mm_P0.65mm, F.Cu at (198.1, 111.4)
- added U12: 74LVCH245APW,118, Package_SO:TSSOP-20_4.4x6.5mm_P0.65mm, F.Cu at (208.3, 111.4)
- added U13: 74LVCH245APW,118, Package_SO:TSSOP-20_4.4x6.5mm_P0.65mm, F.Cu at (231.1, 94.0)
- added U14: 74LVCH245APW,118, Package_SO:TSSOP-20_4.4x6.5mm_P0.65mm, F.Cu at (243.8, 94.0)
- added U15: 74LVCH245APW,118, Package_SO:TSSOP-20_4.4x6.5mm_P0.65mm, F.Cu at (256.2, 94.3)
- added U2: 74LVCH245APW,118, Package_SO:TSSOP-20_4.4x6.5mm_P0.65mm, F.Cu at (83.8, 111.8)
- added U3: 74LVCH245APW,118, Package_SO:TSSOP-20_4.4x6.5mm_P0.65mm, F.Cu at (94.0, 111.8)
- added U4: 74LVCH245APW,118, Package_SO:TSSOP-20_4.4x6.5mm_P0.65mm, F.Cu at (113.0, 111.8)
- added U5: 74LVCH245APW,118, Package_SO:TSSOP-20_4.4x6.5mm_P0.65mm, F.Cu at (123.2, 111.8)
- added U6: 74LVCH245APW,118, Package_SO:TSSOP-20_4.4x6.5mm_P0.65mm, F.Cu at (133.3, 111.8)
- added U7: 74LVCH245APW,118, Package_SO:TSSOP-20_4.4x6.5mm_P0.65mm, F.Cu at (149.9, 111.8)
- added U8: 74LVCH245APW,118, Package_SO:TSSOP-20_4.4x6.5mm_P0.65mm, F.Cu at (160.0, 111.8)
- added U9: 74LVCH245APW,118, Package_SO:TSSOP-20_4.4x6.5mm_P0.65mm, F.Cu at (170.2, 111.8)
Connections:
- J1 pad 10: unconnected-(J1-~{VI6}-Pad10) -> Net-(J1-~{VI6})
- J1 pad 100: unconnected-(J1-GND-Pad100) -> GND
- J1 pad 11: unconnected-(J1-~{VI7}-Pad11) -> Net-(J1-~{VI7})
- J1 pad 12: unconnected-(J1-~{NMI}-Pad12) -> Net-(J1-~{NMI})
- J1 pad 13: unconnected-(J1-~{PWRFAIL}-Pad13) -> Net-(J1-~{PWRFAIL})
- J1 pad 14: unconnected-(J1-~{DMA3}-Pad14) -> Net-(J1-~{DMA3})
- J1 pad 15: unconnected-(J1-A18-Pad15) -> Net-(J1-A18)
- J1 pad 16: unconnected-(J1-A16-Pad16) -> Net-(J1-A16)
- J1 pad 17: unconnected-(J1-A17-Pad17) -> Net-(J1-A17)
- J1 pad 18: unconnected-(J1-~{SDSB}-Pad18) -> Net-(J1-~{SDSB})
- J1 pad 19: unconnected-(J1-~{CDSB}-Pad19) -> Net-(J1-~{CDSB})
- J1 pad 20: unconnected-(J1-GND-Pad20) -> Net-(J3-Pin_11)
- J1 pad 21: unconnected-(J1-NDEF-Pad21) -> Net-(J3-Pin_13)
- J1 pad 22: unconnected-(J1-~{ADBB}-Pad22) -> Net-(J1-~{ADSB})
- J1 pad 23: unconnected-(J1-~{DODSB}-Pad23) -> Net-(J1-~{DODSB})
- J1 pad 24: unconnected-(J1-PHI-Pad24) -> Net-(J1-PHI)
- J1 pad 25: unconnected-(J1-~{pSTVAL}-Pad25) -> Net-(J1-~{pSTVAL})
- J1 pad 26: unconnected-(J1-pHLDA-Pad26) -> Net-(J1-pHLDA)
- J1 pad 27: unconnected-(J1-RFU-Pad27) -> Net-(J4-Pin_1)
- J1 pad 28: unconnected-(J1-RFU-Pad28) -> Net-(J4-Pin_3)
- J1 pad 29: unconnected-(J1-A5-Pad29) -> Net-(J1-A5)
- J1 pad 3: unconnected-(J1-XRDY-Pad3) -> Net-(J1-XRDY)
- J1 pad 30: unconnected-(J1-A4-Pad30) -> Net-(J1-A4)
- J1 pad 31: unconnected-(J1-A3-Pad31) -> Net-(J1-A3)
- J1 pad 32: unconnected-(J1-A15-Pad32) -> Net-(J1-A15)
- J1 pad 33: unconnected-(J1-A12-Pad33) -> Net-(J1-A12)
- J1 pad 34: unconnected-(J1-A9-Pad34) -> Net-(J1-A9)
- J1 pad 35: unconnected-(J1-DO1-Pad35) -> Net-(J1-DO1)
- J1 pad 36: unconnected-(J1-DO0-Pad36) -> Net-(J1-DO0)
- J1 pad 37: unconnected-(J1-A10-Pad37) -> Net-(J1-A10)
- J1 pad 38: unconnected-(J1-DO4-Pad38) -> Net-(J1-DO4)
- J1 pad 39: unconnected-(J1-DO5-Pad39) -> Net-(J1-DO5)
- J1 pad 4: unconnected-(J1-~{VI0}-Pad4) -> Net-(J1-~{VI0})
- J1 pad 40: unconnected-(J1-DO6-Pad40) -> Net-(J1-DO6)
- J1 pad 41: unconnected-(J1-DI2-Pad41) -> Net-(J1-DI2)
- J1 pad 42: unconnected-(J1-DI3-Pad42) -> Net-(J1-DI3)
- J1 pad 43: unconnected-(J1-DI7-Pad43) -> Net-(J1-DI7)
- J1 pad 44: unconnected-(J1-sM1-Pad44) -> Net-(J1-sM1)
- J1 pad 45: unconnected-(J1-sOUT-Pad45) -> Net-(J1-sOUT)
- J1 pad 46: unconnected-(J1-sINP-Pad46) -> Net-(J1-sINP)
- J1 pad 47: unconnected-(J1-sMEMR-Pad47) -> Net-(J1-sMEMR)
- J1 pad 48: unconnected-(J1-sHLTA-Pad48) -> Net-(J1-sHLTA)
- J1 pad 49: unconnected-(J1-CLOCK-Pad49) -> Net-(J1-CLOCK)
- J1 pad 5: unconnected-(J1-~{VI1}-Pad5) -> Net-(J1-~{VI1})
- J1 pad 50: unconnected-(J1-GND-Pad50) -> GND
- J1 pad 53: unconnected-(J1-GND-Pad53) -> Net-(J6-Pin_1)
- J1 pad 54: unconnected-(J1-~{SLV_CLR}-Pad54) -> Net-(J1-~{SLV_CLR})
- J1 pad 55: unconnected-(J1-~{DMA0}-Pad55) -> Net-(J1-~{DMA0})
- J1 pad 56: unconnected-(J1-~{DMA1}-Pad56) -> Net-(J1-~{DMA1})
- J1 pad 57: unconnected-(J1-~{DMA2}-Pad57) -> Net-(J1-~{DMA2})
- J1 pad 58: unconnected-(J1-~{sXTRQ}-Pad58) -> Net-(J1-~{sXTRQ})
- J1 pad 59: unconnected-(J1-A19-Pad59) -> Net-(J1-A19)
- J1 pad 6: unconnected-(J1-~{VI2}-Pad6) -> Net-(J1-~{VI2})
- J1 pad 60: unconnected-(J1-~{SIXTN}-Pad60) -> Net-(J1-~{SIXTN})
- J1 pad 61: unconnected-(J1-A20-Pad61) -> Net-(J1-A20)
- J1 pad 62: unconnected-(J1-A21-Pad62) -> Net-(J1-A21)
- J1 pad 63: unconnected-(J1-A22-Pad63) -> Net-(J1-A22)
- J1 pad 64: unconnected-(J1-A23-Pad64) -> Net-(J1-A23)
- J1 pad 65: unconnected-(J1-NDEF-Pad65) -> Net-(J7-Pin_1)
- J1 pad 66: unconnected-(J1-NDEF-Pad66) -> Net-(J7-Pin_3)
- J1 pad 67: unconnected-(J1-~{PHANTOM}-Pad67) -> Net-(J1-~{PHANTOM})
- J1 pad 68: unconnected-(J1-MWRT-Pad68) -> Net-(J1-MWRT)
- J1 pad 69: unconnected-(J1-RFU-Pad69) -> Net-(J7-Pin_9)
- J1 pad 7: unconnected-(J1-~{VI3}-Pad7) -> Net-(J1-~{VI3})
- J1 pad 70: unconnected-(J1-GND-Pad70) -> Net-(J7-Pin_11)
- J1 pad 71: unconnected-(J1-RFU-Pad71) -> Net-(J7-Pin_13)
- J1 pad 72: unconnected-(J1-RDY-Pad72) -> Net-(J1-RDY)
- J1 pad 73: unconnected-(J1-~{INT}-Pad73) -> Net-(J1-~{INT})
- J1 pad 74: unconnected-(J1-~{HOLD}-Pad74) -> Net-(J1-~{HOLD})
- J1 pad 75: unconnected-(J1-~{RESET}-Pad75) -> Net-(J1-~{RESET})
- J1 pad 76: unconnected-(J1-pSYNC-Pad76) -> Net-(J1-pSYNC)
- J1 pad 77: unconnected-(J1-~{pWR}-Pad77) -> Net-(J1-~{pWR})
- J1 pad 78: unconnected-(J1-pDBIN-Pad78) -> Net-(J1-pDBIN)
- J1 pad 79: unconnected-(J1-A0-Pad79) -> Net-(J1-A0)
- J1 pad 8: unconnected-(J1-~{VI4}-Pad8) -> Net-(J1-~{VI4})
- J1 pad 80: unconnected-(J1-A1-Pad80) -> Net-(J1-A1)
- J1 pad 81: unconnected-(J1-A2-Pad81) -> Net-(J1-A2)
- J1 pad 82: unconnected-(J1-A6-Pad82) -> Net-(J1-A6)
- J1 pad 83: unconnected-(J1-A7-Pad83) -> Net-(J1-A7)
- J1 pad 84: unconnected-(J1-A8-Pad84) -> Net-(J1-A8)
- J1 pad 85: unconnected-(J1-A13-Pad85) -> Net-(J1-A13)
- J1 pad 86: unconnected-(J1-A14-Pad86) -> Net-(J1-A14)
- J1 pad 87: unconnected-(J1-A11-Pad87) -> Net-(J1-A11)
- J1 pad 88: unconnected-(J1-DO2-Pad88) -> Net-(J1-DO2)
- J1 pad 89: unconnected-(J1-DO3-Pad89) -> Net-(J1-DO3)
- J1 pad 9: unconnected-(J1-~{VI5}-Pad9) -> Net-(J1-~{VI5})
- J1 pad 90: unconnected-(J1-DO7-Pad90) -> Net-(J1-DO7)
- J1 pad 91: unconnected-(J1-DI4-Pad91) -> Net-(J1-DI4)
- J1 pad 92: unconnected-(J1-DI5-Pad92) -> Net-(J1-DI5)
- J1 pad 93: unconnected-(J1-DI6-Pad93) -> Net-(J1-DI6)
- J1 pad 94: unconnected-(J1-DI1-Pad94) -> Net-(J1-DI1)
- J1 pad 95: unconnected-(J1-DI0-Pad95) -> Net-(J1-DI0)
- J1 pad 96: unconnected-(J1-sINTA-Pad96) -> Net-(J1-sINTA)
- J1 pad 97: unconnected-(J1-~{sWO}-Pad97) -> Net-(J1-~{sWO})
- J1 pad 98: unconnected-(J1-~{ERROR}-Pad98) -> Net-(J1-~{ERROR})
- J1 pad 99: unconnected-(J1-~{POC}-Pad99) -> Net-(J1-~{POC})
Routing:
- net Net-(A1-GPIO2): track 0.00 -> 125.4 mm
- net Net-(A1-GPIO3): track 0.00 -> 121.3 mm
- net Net-(A1-GPIO4): track 0.00 -> 116.4 mm
- net Net-(A1-GPIO5): track 0.00 -> 112.8 mm
- net Net-(A1-GPIO6): track 0.00 -> 101.5 mm
- net Net-(A1-GPIO7): track 0.00 -> 96.6 mm
- net Net-(A1-GPIO8): track 0.00 -> 91.7 mm
- net Net-(A1-GPIO9): track 0.00 -> 86.8 mm
- net Net-(A1-GPIO10): track 0.00 -> 78.9 mm
- net Net-(A1-GPIO28_ADC2): track 0.00 -> 73.1 mm
- net Net-(A1-GPIO27_ADC1): track 0.00 -> 67.1 mm
- net Net-(A1-GPIO26_ADC0): track 0.00 -> 64.1 mm
- net Net-(A1-GPIO22): track 0.00 -> 57.5 mm
- net Net-(A1-GPIO11): track 0.00 -> 55.5 mm
- net Net-(A1-GPIO12): track 0.00 -> 52.9 mm
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Other:
- board text added: "11"
- board text added: "12"
- board text added: "13"
- board text added: "14"
- board text added: "15"
- board text added: "16"
- board text added: "17"
- board text added: "18"
- board text added: "19"
- board text added: "21"
- board text added: "22"
- board text added: "23"
- board text added: "24"
- board text added: "25"
- board text added: "26"
- board text added: "27"
- board text added: "3"
- board text added: "39"
- board text added: "4"
- board text added: "5"
- board text added: "53"
- board text added: "54"
- board text added: "55"
- board text added: "56"
- board text added: "57"
- board text added: "58"
- board text added: "59"
- board text added: "6"
- board text added: "61"
- board text added: "62"
- board text added: "63"
- board text added: "64"
- board text added: "65"
- board text added: "66"
- board text added: "67"
- board text added: "68"
- board text added: "69"
- board text added: "7"
- board text added: "71"
- board text added: "72"
- board text added: "73"
- board text added: "74"
- board text added: "75"
- board text added: "76"
- board text added: "77"
- board text added: "8"
- board text added: "9"
- board text added: "A16"
- board text added: "A17"
- board text added: "A18"
- board text added: "A19"
- board text added: "A20"
- board text added: "A21"
- board text added: "A22"
- board text added: "A23"
- board text added: "GND"
- board text added: "MWRT"
- board text added: "NDEF"
- board text added: "PSI"
- board text added: "RDY"
- board text added: "XRDY"
- board text added: "pHLDA"
- board text added: "~{ADSB}"
- board text added: "~{CDSB}"
- board text added: "~{DMA0}"
- board text added: "~{DMA1}"
- board text added: "~{DMA2}"
- board text added: "~{DMA3}"
- board text added: "~{DODSB}"
- board text added: "~{HOLD}"
- board text added: "~{INT}"
- board text added: "~{NMI}"
- board text added: "~{PHANTOM}"
- board text added: "~{PWRFAIL}"
- board text added: "~{RESET}"
- board text added: "~{SDSB}"
- board text added: "~{SLV_CLR}"
- board text added: "~{SXTN}"
- board text added: "~{VI0}"
- board text added: "~{VI1}"
- board text added: "~{VI2}"
- board text added: "~{VI3}"
- board text added: "~{VI4}"
- board text added: "~{VI5}"
- board text added: "~{VI6}"
- board text added: "~{VI7}"
- board text added: "~{pSTVAL}"
- board text added: "~{pSYNC}"
- board text added: "~{sXTRQ}"

Commit message: Add S100 power
Parts:
- added C31: .1uF, Capacitor_SMD:C_0603_1608Metric_Pad1.08x0.95mm_HandSolder, F.Cu at (36.6, 94.4)
- added C33: 47pF, Capacitor_SMD:C_0603_1608Metric_Pad1.08x0.95mm_HandSolder, F.Cu at (36.6, 96.9)
- added C47: 10uF, Capacitor_SMD:C_0805_2012Metric_Pad1.18x1.45mm_HandSolder, F.Cu at (32.0, 94.6)
- added C50: 22uF, Capacitor_SMD:C_0805_2012Metric_Pad1.18x1.45mm_HandSolder, F.Cu at (32.0, 97.7)
- added C58: 22uF, Capacitor_SMD:C_0805_2012Metric_Pad1.18x1.45mm_HandSolder, F.Cu at (32.0, 100.7)
- added C66: 22uF, Capacitor_SMD:C_0805_2012Metric_Pad1.18x1.45mm_HandSolder, F.Cu at (32.0, 103.7)
- added C67: 22uF, Capacitor_SMD:C_0805_2012Metric_Pad1.18x1.45mm_HandSolder, F.Cu at (32.0, 106.7)
- added D4: SS56F, Diode_SMD:D_SMB_Handsoldering, F.Cu at (43.0, 109.2)
- added L11: 6.8uH, Inductor_SMD:L_Bourns-SRN6028, F.Cu at (38.3, 119.9)
- added R1: 1K, Resistor_SMD:R_0603_1608Metric_Pad0.98x0.95mm_HandSolder, F.Cu at (50.8, 38.1)
- added R2: 1K, Resistor_SMD:R_0603_1608Metric_Pad0.98x0.95mm_HandSolder, F.Cu at (48.3, 38.1)
- added R3: 1K, Resistor_SMD:R_0603_1608Metric_Pad0.98x0.95mm_HandSolder, F.Cu at (53.3, 38.1)
- added R47: 8K4, Resistor_SMD:R_0603_1608Metric_Pad0.98x0.95mm_HandSolder, F.Cu at (29.6, 116.9)
- added R48: 1K6, Resistor_SMD:R_0603_1608Metric_Pad0.98x0.95mm_HandSolder, F.Cu at (29.6, 119.4)
- added U16: AP63300, Package_TO_SOT_SMD:SOT-23-6, F.Cu at (37.0, 126.0)
Connections:
- net /VSYS renamed +VSYS
- A1 pad 36: unconnected-(A1-3V3-Pad36) -> Net-(A1-3V3)
- A4 pad 36: unconnected-(A4-3V3-Pad36) -> Net-(A4-3V3)
- D1 pad 1: unconnected-(D1-K-Pad1) -> GND
- D1 pad 2: unconnected-(D1-A-Pad2) -> Net-(D1-A)
- D2 pad 1: unconnected-(D2-K-Pad1) -> GND
- D2 pad 2: unconnected-(D2-A-Pad2) -> Net-(D2-A)
- D3 pad 1: unconnected-(D3-K-Pad1) -> GND
- D3 pad 2: unconnected-(D3-A-Pad2) -> Net-(D3-A)
- J1 pad 1: unconnected-(J1-+8-Pad1) -> +S100_8V
- J1 pad 51: unconnected-(J1-+8-Pad51) -> +S100_8V
- U1 pad 20: unconnected-(U1-VCC-Pad20) -> Net-(A1-3V3)
- U10 pad 20: unconnected-(U10-VCC-Pad20) -> Net-(A4-3V3)
- U11 pad 20: unconnected-(U11-VCC-Pad20) -> Net-(A4-3V3)
- U12 pad 20: unconnected-(U12-VCC-Pad20) -> Net-(A4-3V3)
- U2 pad 20: unconnected-(U2-VCC-Pad20) -> Net-(A1-3V3)
- U3 pad 20: unconnected-(U3-VCC-Pad20) -> Net-(A1-3V3)

Commit message: Checkpoint
Parts:
- added C1: .1uF, Capacitor_SMD:C_0603_1608Metric_Pad1.08x0.95mm_HandSolder, F.Cu at (69.3, 109.5)
- added C10: .1uF, Capacitor_SMD:C_0603_1608Metric_Pad1.08x0.95mm_HandSolder, F.Cu at (182.9, 109.2)
- added C11: .1uF, Capacitor_SMD:C_0603_1608Metric_Pad1.08x0.95mm_HandSolder, F.Cu at (193.8, 109.4)
- added C12: .1uF, Capacitor_SMD:C_0603_1608Metric_Pad1.08x0.95mm_HandSolder, F.Cu at (204.0, 109.2)
- added C13: .1uF, Capacitor_SMD:C_0603_1608Metric_Pad1.08x0.95mm_HandSolder, F.Cu at (226.6, 91.8)
- added C14: .1uF, Capacitor_SMD:C_0603_1608Metric_Pad1.08x0.95mm_HandSolder, F.Cu at (239.3, 91.9)
- added C15: .1uF, Capacitor_SMD:C_0603_1608Metric_Pad1.08x0.95mm_HandSolder, F.Cu at (252.2, 91.8)
- added C2: .1uF, Capacitor_SMD:C_0603_1608Metric_Pad1.08x0.95mm_HandSolder, F.Cu at (79.5, 109.2)
- added C3: .1uF, Capacitor_SMD:C_0603_1608Metric_Pad1.08x0.95mm_HandSolder, F.Cu at (89.7, 109.5)
- added C4: .1uF, Capacitor_SMD:C_0603_1608Metric_Pad1.08x0.95mm_HandSolder, F.Cu at (108.7, 109.9)
- added C5: .1uF, Capacitor_SMD:C_0603_1608Metric_Pad1.08x0.95mm_HandSolder, F.Cu at (118.9, 109.5)
- added C6: .1uF, Capacitor_SMD:C_0603_1608Metric_Pad1.08x0.95mm_HandSolder, F.Cu at (129.0, 109.5)
- added C7: .1uF, Capacitor_SMD:C_0603_1608Metric_Pad1.08x0.95mm_HandSolder, F.Cu at (145.5, 109.7)
- added C8: .1uF, Capacitor_SMD:C_0603_1608Metric_Pad1.08x0.95mm_HandSolder, F.Cu at (155.7, 109.5)
- added C9: .1uF, Capacitor_SMD:C_0603_1608Metric_Pad1.08x0.95mm_HandSolder, F.Cu at (165.9, 109.7)
- added D5: SS56F, Diode_SMD:D_SMB_Handsoldering, F.Cu at (205.7, 39.4)
- added J12: USB4105-GF-A, Connector_USB:USB_C_Receptacle_GCT_USB4105-xx-A_16P_TopMnt_Horizontal, F.Cu at (199.5, 29.1)
- added J13: Conn_01x01, Connector_PinHeader_2.54mm:PinHeader_1x01_P2.54mm_Vertical, F.Cu at (120.9, 130.0)
- added J14: Conn_01x01, Connector_PinHeader_2.54mm:PinHeader_1x01_P2.54mm_Vertical, F.Cu at (120.9, 146.3)
- added J15: Conn_01x02, Connector_PinHeader_2.54mm:PinHeader_1x02_P2.54mm_Vertical, F.Cu at (210.8, 27.9)
- added J16: Conn_01x02, Connector_PinHeader_2.54mm:PinHeader_1x02_P2.54mm_Vertical, F.Cu at (163.8, 27.9)
- added J17: Conn_01x02, Connector_PinHeader_2.54mm:PinHeader_1x02_P2.54mm_Vertical, F.Cu at (128.3, 27.9)
- added J18: Conn_01x02, Connector_PinHeader_2.54mm:PinHeader_1x02_P2.54mm_Vertical, F.Cu at (92.7, 27.9)
- added J19: Conn_01x02, Connector_PinHeader_2.54mm:PinHeader_1x02_P2.54mm_Vertical, F.Cu at (57.1, 27.9)
- added R10: 1K, Resistor_SMD:R_0603_1608Metric_Pad0.98x0.95mm_HandSolder, F.Cu at (239.3, 95.9)
- added R4: 5K1, Resistor_SMD:R_0603_1608Metric_Pad0.98x0.95mm_HandSolder, F.Cu at (198.1, 38.1)
- added R5: 5K1, Resistor_SMD:R_0603_1608Metric_Pad0.98x0.95mm_HandSolder, F.Cu at (200.7, 38.1)
- added R6: 1K, Resistor_SMD:R_0603_1608Metric_Pad0.98x0.95mm_HandSolder, F.Cu at (79.5, 113.8)
- added R7: 1K, Resistor_SMD:R_0603_1608Metric_Pad0.98x0.95mm_HandSolder, F.Cu at (118.9, 113.9)
- added R8: 1K, Resistor_SMD:R_0603_1608Metric_Pad0.98x0.95mm_HandSolder, F.Cu at (155.7, 114.0)
- added R9: 1K, Resistor_SMD:R_0603_1608Metric_Pad0.98x0.95mm_HandSolder, F.Cu at (193.8, 113.5)
- added SW1: SW_MEC_5E, S100-footprints:tactile, F.Cu at (242.2, 29.2)
- added U17: LM7805_TO220, Package_TO_SOT_THT:TO-220-3_Horizontal_TabDown, F.Cu at (35.8, 113.4)
- H1, H2: value MountingHole -> Card Ejector
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Connections:
- A1 pad 13: Net-(A1-GND-Pad13) -> GND
- A1 pad 18: Net-(A1-GND-Pad13) -> GND
- A1 pad 23: Net-(A1-GND-Pad13) -> GND
- A1 pad 28: Net-(A1-GND-Pad13) -> GND
- A1 pad 3: Net-(A1-GND-Pad13) -> GND
- A1 pad 30: unconnected-(A1-RUN-Pad30) -> /~{PICO_RESET}
- A1 pad 33: unconnected-(A1-AGND-Pad33) -> GND
- A1 pad 38: Net-(A1-GND-Pad13) -> GND
- A1 pad 8: Net-(A1-GND-Pad13) -> GND
- A2 pad 1: unconnected-(A2-GPIO0-Pad1) -> Net-(A2-GPIO0)
- A2 pad 10: unconnected-(A2-GPIO7-Pad10) -> Net-(A2-GPIO7)
- A2 pad 11: unconnected-(A2-GPIO8-Pad11) -> Net-(A2-GPIO8)
- A2 pad 12: unconnected-(A2-GPIO9-Pad12) -> Net-(A2-GPIO9)
- A2 pad 13: Net-(A2-GND-Pad13) -> GND
- A2 pad 14: unconnected-(A2-GPIO10-Pad14) -> Net-(A2-GPIO10)
- A2 pad 15: unconnected-(A2-GPIO11-Pad15) -> Net-(A2-GPIO11)
- A2 pad 16: unconnected-(A2-GPIO12-Pad16) -> Net-(A2-GPIO12)
- A2 pad 17: unconnected-(A2-GPIO13-Pad17) -> Net-(A2-GPIO13)
- A2 pad 18: Net-(A2-GND-Pad13) -> GND
- A2 pad 19: unconnected-(A2-GPIO14-Pad19) -> Net-(A2-GPIO14)
- A2 pad 2: unconnected-(A2-GPIO1-Pad2) -> Net-(A2-GPIO0)
- A2 pad 20: unconnected-(A2-GPIO15-Pad20) -> Net-(A2-GPIO15)
- A2 pad 21: unconnected-(A2-GPIO16-Pad21) -> Net-(A2-GPIO16)
- A2 pad 22: unconnected-(A2-GPIO17-Pad22) -> Net-(A2-GPIO17)
- A2 pad 23: Net-(A2-GND-Pad13) -> GND
- A2 pad 24: unconnected-(A2-GPIO18-Pad24) -> Net-(A2-GPIO18)
- A2 pad 25: unconnected-(A2-GPIO19-Pad25) -> Net-(A2-GPIO19)
- A2 pad 26: unconnected-(A2-GPIO20-Pad26) -> Net-(A2-GPIO20)
- A2 pad 27: unconnected-(A2-GPIO21-Pad27) -> Net-(A2-GPIO21)
- A2 pad 28: Net-(A2-GND-Pad13) -> GND
- A2 pad 29: unconnected-(A2-GPIO22-Pad29) -> Net-(A2-GPIO22)
- A2 pad 3: Net-(A2-GND-Pad13) -> GND
- A2 pad 30: unconnected-(A2-RUN-Pad30) -> /~{PICO_RESET}
- A2 pad 31: unconnected-(A2-GPIO26_ADC0-Pad31) -> Net-(A2-GPIO26_ADC0)
- A2 pad 32: unconnected-(A2-GPIO27_ADC1-Pad32) -> Net-(A2-GPIO27_ADC1)
- A2 pad 33: unconnected-(A2-AGND-Pad33) -> GND
- A2 pad 34: unconnected-(A2-GPIO28_ADC2-Pad34) -> Net-(A2-GPIO28_ADC2)
- A2 pad 36: unconnected-(A2-3V3-Pad36) -> Net-(A2-3V3)
- A2 pad 38: Net-(A2-GND-Pad13) -> GND
- A2 pad 4: unconnected-(A2-GPIO2-Pad4) -> Net-(A2-GPIO2)
- A2 pad 5: unconnected-(A2-GPIO3-Pad5) -> Net-(A2-GPIO3)
- A2 pad 6: unconnected-(A2-GPIO4-Pad6) -> Net-(A2-GPIO4)
- A2 pad 7: unconnected-(A2-GPIO5-Pad7) -> Net-(A2-GPIO5)
- A2 pad 8: Net-(A2-GND-Pad13) -> GND
- A2 pad 9: unconnected-(A2-GPIO6-Pad9) -> Net-(A2-GPIO6)
- A3 pad 1: unconnected-(A3-GPIO0-Pad1) -> Net-(A3-GPIO0)
- A3 pad 10: unconnected-(A3-GPIO7-Pad10) -> Net-(A3-GPIO7)
- A3 pad 11: unconnected-(A3-GPIO8-Pad11) -> Net-(A3-GPIO8)
- A3 pad 12: unconnected-(A3-GPIO9-Pad12) -> Net-(A3-GPIO9)
- A3 pad 13: Net-(A3-GND-Pad13) -> GND
- A3 pad 14: unconnected-(A3-GPIO10-Pad14) -> Net-(A3-GPIO10)
- A3 pad 15: unconnected-(A3-GPIO11-Pad15) -> Net-(A3-GPIO11)
- A3 pad 16: unconnected-(A3-GPIO12-Pad16) -> Net-(A3-GPIO12)
- A3 pad 17: unconnected-(A3-GPIO13-Pad17) -> Net-(A3-GPIO13)
- A3 pad 18: Net-(A3-GND-Pad13) -> GND
- A3 pad 19: unconnected-(A3-GPIO14-Pad19) -> Net-(A3-GPIO14)
- A3 pad 2: unconnected-(A3-GPIO1-Pad2) -> Net-(A3-GPIO0)
- A3 pad 20: unconnected-(A3-GPIO15-Pad20) -> Net-(A3-GPIO15)
- A3 pad 21: unconnected-(A3-GPIO16-Pad21) -> Net-(A3-GPIO16)
- A3 pad 22: unconnected-(A3-GPIO17-Pad22) -> Net-(A3-GPIO17)
- A3 pad 23: Net-(A3-GND-Pad13) -> GND
- A3 pad 24: unconnected-(A3-GPIO18-Pad24) -> Net-(A3-GPIO18)
- A3 pad 25: unconnected-(A3-GPIO19-Pad25) -> Net-(A3-GPIO19)
- A3 pad 26: unconnected-(A3-GPIO20-Pad26) -> Net-(A3-GPIO20)
- A3 pad 27: unconnected-(A3-GPIO21-Pad27) -> Net-(A3-GPIO21)
- A3 pad 28: Net-(A3-GND-Pad13) -> GND
- A3 pad 29: unconnected-(A3-GPIO22-Pad29) -> Net-(A3-GPIO22)
- A3 pad 3: Net-(A3-GND-Pad13) -> GND
- A3 pad 30: unconnected-(A3-RUN-Pad30) -> /~{PICO_RESET}
- A3 pad 31: unconnected-(A3-GPIO26_ADC0-Pad31) -> Net-(A3-GPIO26_ADC0)
- A3 pad 32: unconnected-(A3-GPIO27_ADC1-Pad32) -> Net-(A3-GPIO27_ADC1)
- A3 pad 33: unconnected-(A3-AGND-Pad33) -> GND
- A3 pad 34: unconnected-(A3-GPIO28_ADC2-Pad34) -> Net-(A3-GPIO28_ADC2)
- A3 pad 36: unconnected-(A3-3V3-Pad36) -> Net-(A3-3V3)
- A3 pad 38: Net-(A3-GND-Pad13) -> GND
- A3 pad 4: unconnected-(A3-GPIO2-Pad4) -> Net-(A3-GPIO2)
- A3 pad 5: unconnected-(A3-GPIO3-Pad5) -> Net-(A3-GPIO3)
- A3 pad 6: unconnected-(A3-GPIO4-Pad6) -> Net-(A3-GPIO4)
- A3 pad 7: unconnected-(A3-GPIO5-Pad7) -> Net-(A3-GPIO5)
- A3 pad 8: Net-(A3-GND-Pad13) -> GND
- A3 pad 9: unconnected-(A3-GPIO6-Pad9) -> Net-(A3-GPIO6)
- A4 pad 1: unconnected-(A4-GPIO0-Pad1) -> Net-(A4-GPIO0)
- A4 pad 10: unconnected-(A4-GPIO7-Pad10) -> Net-(A4-GPIO7)
- A4 pad 11: unconnected-(A4-GPIO8-Pad11) -> Net-(A4-GPIO8)
- A4 pad 12: unconnected-(A4-GPIO9-Pad12) -> Net-(A4-GPIO9)
- A4 pad 13: Net-(A4-GND-Pad13) -> GND
- A4 pad 14: unconnected-(A4-GPIO10-Pad14) -> Net-(A4-GPIO10)
- A4 pad 15: unconnected-(A4-GPIO11-Pad15) -> Net-(A4-GPIO11)
- A4 pad 16: unconnected-(A4-GPIO12-Pad16) -> Net-(A4-GPIO12)
- A4 pad 17: unconnected-(A4-GPIO13-Pad17) -> Net-(A4-GPIO13)
- A4 pad 18: Net-(A4-GND-Pad13) -> GND
- A4 pad 19: unconnected-(A4-GPIO14-Pad19) -> Net-(A4-GPIO14)
- A4 pad 2: unconnected-(A4-GPIO1-Pad2) -> Net-(A4-GPIO0)
- A4 pad 20: unconnected-(A4-GPIO15-Pad20) -> Net-(A4-GPIO15)
- A4 pad 21: unconnected-(A4-GPIO16-Pad21) -> Net-(A4-GPIO16)
- A4 pad 22: unconnected-(A4-GPIO17-Pad22) -> Net-(A4-GPIO17)
- A4 pad 23: Net-(A4-GND-Pad13) -> GND
- A4 pad 24: unconnected-(A4-GPIO18-Pad24) -> Net-(A4-GPIO18)
- A4 pad 25: unconnected-(A4-GPIO19-Pad25) -> Net-(A4-GPIO19)
- A4 pad 26: unconnected-(A4-GPIO20-Pad26) -> Net-(A4-GPIO20)
- A4 pad 27: unconnected-(A4-GPIO21-Pad27) -> Net-(A4-GPIO21)
- A4 pad 28: Net-(A4-GND-Pad13) -> GND
- A4 pad 29: unconnected-(A4-GPIO22-Pad29) -> Net-(A4-GPIO22)
- A4 pad 3: Net-(A4-GND-Pad13) -> GND
- A4 pad 30: unconnected-(A4-RUN-Pad30) -> /~{PICO_RESET}
- A4 pad 31: unconnected-(A4-GPIO26_ADC0-Pad31) -> Net-(A4-GPIO26_ADC0)
- A4 pad 32: unconnected-(A4-GPIO27_ADC1-Pad32) -> Net-(A4-GPIO27_ADC1)
- A4 pad 33: unconnected-(A4-AGND-Pad33) -> GND
- A4 pad 34: unconnected-(A4-GPIO28_ADC2-Pad34) -> Net-(A4-GPIO28_ADC2)
- A4 pad 38: Net-(A4-GND-Pad13) -> GND
- A4 pad 4: unconnected-(A4-GPIO2-Pad4) -> Net-(A4-GPIO2)
- A4 pad 5: unconnected-(A4-GPIO3-Pad5) -> Net-(A4-GPIO3)
- A4 pad 6: unconnected-(A4-GPIO4-Pad6) -> Net-(A4-GPIO4)
- A4 pad 7: unconnected-(A4-GPIO5-Pad7) -> Net-(A4-GPIO5)
- A4 pad 8: Net-(A4-GND-Pad13) -> GND
- A4 pad 9: unconnected-(A4-GPIO6-Pad9) -> Net-(A4-GPIO6)
- A5 pad 1: unconnected-(A5-GPIO0-Pad1) -> Net-(A5-GPIO0)
- A5 pad 10: unconnected-(A5-GPIO7-Pad10) -> Net-(A5-GPIO7)
- A5 pad 11: unconnected-(A5-GPIO8-Pad11) -> Net-(A5-GPIO8)
- A5 pad 12: unconnected-(A5-GPIO9-Pad12) -> Net-(A5-GPIO9)
- A5 pad 13: Net-(A5-GND-Pad13) -> GND
- A5 pad 14: unconnected-(A5-GPIO10-Pad14) -> Net-(A5-GPIO10)
- A5 pad 15: unconnected-(A5-GPIO11-Pad15) -> Net-(A5-GPIO11)
- A5 pad 16: unconnected-(A5-GPIO12-Pad16) -> Net-(A5-GPIO12)
- A5 pad 17: unconnected-(A5-GPIO13-Pad17) -> Net-(A5-GPIO13)
- A5 pad 18: Net-(A5-GND-Pad13) -> GND
- A5 pad 19: unconnected-(A5-GPIO14-Pad19) -> Net-(A5-GPIO14)
- A5 pad 2: unconnected-(A5-GPIO1-Pad2) -> Net-(A5-GPIO0)
- A5 pad 20: unconnected-(A5-GPIO15-Pad20) -> Net-(A5-GPIO15)
- A5 pad 21: unconnected-(A5-GPIO16-Pad21) -> Net-(A5-GPIO16)
- A5 pad 22: unconnected-(A5-GPIO17-Pad22) -> Net-(A5-GPIO17)
- A5 pad 23: Net-(A5-GND-Pad13) -> GND
- A5 pad 24: unconnected-(A5-GPIO18-Pad24) -> Net-(A5-GPIO18)
- A5 pad 25: unconnected-(A5-GPIO19-Pad25) -> Net-(A5-GPIO19)
- A5 pad 26: unconnected-(A5-GPIO20-Pad26) -> Net-(A5-GPIO20)
- A5 pad 27: unconnected-(A5-GPIO21-Pad27) -> Net-(A5-GPIO21)
- A5 pad 28: Net-(A5-GND-Pad13) -> GND
- A5 pad 29: unconnected-(A5-GPIO22-Pad29) -> Net-(A5-GPIO22)
- A5 pad 3: Net-(A5-GND-Pad13) -> GND
- A5 pad 31: unconnected-(A5-GPIO26_ADC0-Pad31) -> Net-(A5-GPIO26_ADC0)
- A5 pad 32: unconnected-(A5-GPIO27_ADC1-Pad32) -> Net-(A5-GPIO27_ADC1)
- A5 pad 33: unconnected-(A5-AGND-Pad33) -> GND
- A5 pad 34: unconnected-(A5-GPIO28_ADC2-Pad34) -> Net-(A5-GPIO28_ADC2)
- A5 pad 38: Net-(A5-GND-Pad13) -> GND
- A5 pad 4: unconnected-(A5-GPIO2-Pad4) -> Net-(A5-GPIO2)
- A5 pad 5: unconnected-(A5-GPIO3-Pad5) -> Net-(A5-GPIO3)
- A5 pad 6: unconnected-(A5-GPIO4-Pad6) -> Net-(A5-GPIO4)
- A5 pad 7: unconnected-(A5-GPIO5-Pad7) -> Net-(A5-GPIO5)
- A5 pad 8: Net-(A5-GND-Pad13) -> GND
- A5 pad 9: unconnected-(A5-GPIO6-Pad9) -> Net-(A5-GPIO6)
- J10 pad 1: unconnected-(J10-Pin_1-Pad1) -> /T1
- J10 pad 10: unconnected-(J10-Pin_10-Pad10) -> /T9
- J10 pad 11: unconnected-(J10-Pin_11-Pad11) -> /T11
- J10 pad 12: unconnected-(J10-Pin_12-Pad12) -> /T11
- J10 pad 13: unconnected-(J10-Pin_13-Pad13) -> /T13
- J10 pad 14: unconnected-(J10-Pin_14-Pad14) -> /T13
- J10 pad 15: unconnected-(J10-Pin_15-Pad15) -> /T15
- J10 pad 16: unconnected-(J10-Pin_16-Pad16) -> /T15
- J10 pad 17: unconnected-(J10-Pin_17-Pad17) -> /T17
- J10 pad 18: unconnected-(J10-Pin_18-Pad18) -> /T17
- J10 pad 19: unconnected-(J10-Pin_19-Pad19) -> /T19
- J10 pad 2: unconnected-(J10-Pin_2-Pad2) -> /T1
- J10 pad 20: unconnected-(J10-Pin_20-Pad20) -> /T19
- J10 pad 21: unconnected-(J10-Pin_21-Pad21) -> /T21
- J10 pad 22: unconnected-(J10-Pin_22-Pad22) -> /T21
- J10 pad 23: unconnected-(J10-Pin_23-Pad23) -> /T23
- J10 pad 24: unconnected-(J10-Pin_24-Pad24) -> /T23
- J10 pad 25: unconnected-(J10-Pin_25-Pad25) -> GND
- J10 pad 26: unconnected-(J10-Pin_26-Pad26) -> GND
- J10 pad 3: unconnected-(J10-Pin_3-Pad3) -> /T3
- J10 pad 4: unconnected-(J10-Pin_4-Pad4) -> /T3
- J10 pad 5: unconnected-(J10-Pin_5-Pad5) -> /T5
- J10 pad 6: unconnected-(J10-Pin_6-Pad6) -> /T5
- J10 pad 7: unconnected-(J10-Pin_7-Pad7) -> /T7
- J10 pad 8: unconnected-(J10-Pin_8-Pad8) -> /T7
- J10 pad 9: unconnected-(J10-Pin_9-Pad9) -> /T9
- J11 pad 1: unconnected-(J11-Pin_1-Pad1) -> /T2
- J11 pad 10: unconnected-(J11-Pin_10-Pad10) -> /T10
- J11 pad 11: unconnected-(J11-Pin_11-Pad11) -> /T12
- J11 pad 12: unconnected-(J11-Pin_12-Pad12) -> /T12
- J11 pad 13: unconnected-(J11-Pin_13-Pad13) -> /T14
- J11 pad 14: unconnected-(J11-Pin_14-Pad14) -> /T14
- J11 pad 15: unconnected-(J11-Pin_15-Pad15) -> /T16
- J11 pad 16: unconnected-(J11-Pin_16-Pad16) -> /T16
- J11 pad 17: unconnected-(J11-Pin_17-Pad17) -> /T18
- J11 pad 18: unconnected-(J11-Pin_18-Pad18) -> /T18
- J11 pad 19: unconnected-(J11-Pin_19-Pad19) -> /T20
- J11 pad 2: unconnected-(J11-Pin_2-Pad2) -> /T2
- J11 pad 20: unconnected-(J11-Pin_20-Pad20) -> /T20
- J11 pad 21: unconnected-(J11-Pin_21-Pad21) -> /T22
- J11 pad 22: unconnected-(J11-Pin_22-Pad22) -> /T22
- J11 pad 23: unconnected-(J11-Pin_23-Pad23) -> /T24
- J11 pad 24: unconnected-(J11-Pin_24-Pad24) -> /T24
- J11 pad 25: unconnected-(J11-Pin_25-Pad25) -> GND
- J11 pad 26: unconnected-(J11-Pin_26-Pad26) -> GND
- J11 pad 3: unconnected-(J11-Pin_3-Pad3) -> /T4
- J11 pad 4: unconnected-(J11-Pin_4-Pad4) -> /T4
- J11 pad 5: unconnected-(J11-Pin_5-Pad5) -> /T6
- J11 pad 6: unconnected-(J11-Pin_6-Pad6) -> /T6
- J11 pad 7: unconnected-(J11-Pin_7-Pad7) -> /T8
- J11 pad 8: unconnected-(J11-Pin_8-Pad8) -> /T8
- J11 pad 9: unconnected-(J11-Pin_9-Pad9) -> /T10
- J2 pad 20: /~{INT} -> /~{NMI}
- J5 pad 24: unconnected-(J5-Pin_24-Pad24) -> /A4.23
- J9 pad 24: unconnected-(J9-Pin_24-Pad24) -> /A4.24
- R1 pad 1: unconnected-(R1-Pad1) -> +S100_5V
- R1 pad 2: Net-(D2-A) -> Net-(D1-A)
- R2 pad 1: unconnected-(R2-Pad1) -> +VSYS
- R2 pad 2: Net-(D3-A) -> Net-(D2-A)
- R3 pad 1: +S100_5V -> +USBC5
- R3 pad 2: Net-(D1-A) -> Net-(D3-A)
- U1 pad 1: GND -> Net-(U1-DIR)
- U1 pad 10: unconnected-(U1-GND-Pad10) -> GND
- U10 pad 1: unconnected-(U10-DIR-Pad1) -> Net-(U10-DIR)
- U10 pad 10: unconnected-(U10-GND-Pad10) -> GND
- U10 pad 11: unconnected-(U10-B8-Pad11) -> Net-(A4-GPIO9)
- U10 pad 12: unconnected-(U10-B7-Pad12) -> Net-(A4-GPIO8)
- U10 pad 13: unconnected-(U10-B6-Pad13) -> Net-(A4-GPIO7)
- U10 pad 14: unconnected-(U10-B5-Pad14) -> Net-(A4-GPIO6)
- U10 pad 15: unconnected-(U10-B4-Pad15) -> Net-(A4-GPIO5)
- U10 pad 16: unconnected-(U10-B3-Pad16) -> Net-(A4-GPIO4)
- U10 pad 17: unconnected-(U10-B2-Pad17) -> Net-(A4-GPIO3)
- U10 pad 18: unconnected-(U10-B1-Pad18) -> Net-(A4-GPIO2)
- U10 pad 19: unconnected-(U10-~{OE}-Pad19) -> GND
- U10 pad 2: unconnected-(U10-A1-Pad2) -> /DO5
- U10 pad 3: unconnected-(U10-A2-Pad3) -> /DO3
- U10 pad 4: unconnected-(U10-A3-Pad4) -> /DO6
- U10 pad 5: unconnected-(U10-A4-Pad5) -> /DO7
- U10 pad 6: unconnected-(U10-A5-Pad6) -> /DI2
- U10 pad 7: unconnected-(U10-A6-Pad7) -> /DI4
- U10 pad 8: unconnected-(U10-A7-Pad8) -> /DI3
- U10 pad 9: unconnected-(U10-A8-Pad9) -> /DI5
- U11 pad 1: unconnected-(U11-DIR-Pad1) -> Net-(U10-DIR)
- U11 pad 10: unconnected-(U11-GND-Pad10) -> GND
- U11 pad 11: unconnected-(U11-B8-Pad11) -> Net-(A4-GPIO17)
- U11 pad 12: unconnected-(U11-B7-Pad12) -> Net-(A4-GPIO16)
- U11 pad 13: unconnected-(U11-B6-Pad13) -> Net-(A4-GPIO15)
- U11 pad 14: unconnected-(U11-B5-Pad14) -> Net-(A4-GPIO14)
- U11 pad 15: unconnected-(U11-B4-Pad15) -> Net-(A4-GPIO13)
- U11 pad 16: unconnected-(U11-B3-Pad16) -> Net-(A4-GPIO12)
- U11 pad 17: unconnected-(U11-B2-Pad17) -> Net-(A4-GPIO11)
- U11 pad 18: unconnected-(U11-B1-Pad18) -> Net-(A4-GPIO10)
- U11 pad 19: unconnected-(U11-~{OE}-Pad19) -> GND
- U11 pad 2: unconnected-(U11-A1-Pad2) -> /DI7
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Routing:
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- added copper zone on In2.Cu, net +VSYS
- added copper zone on B.Cu, net GND
- added copper zone on F.Cu, net GND
- added copper zone on In1.Cu, net GND
Other:
- copper layers 2 -> 4
- board text added: "2"
- board text added: "28"
- board text added: "29"
- board text added: "31"
- board text added: "32"
- board text added: "33"
- board text added: "34"
- board text added: "35"
- board text added: "36"
- board text added: "37"
- board text added: "38"
- board text added: "41"
- board text added: "42"
- board text added: "43"
- board text added: "44"
- board text added: "45"
- board text added: "46"
- board text added: "47"
- board text added: "48"
- board text added: "49"
- board text added: "78"
- board text added: "79"
- board text added: "81"
- board text added: "82"
- board text added: "83"
- board text added: "84"
- board text added: "85"
- board text added: "86"
- board text added: "87"
- board text added: "88"
- board text added: "89"
- board text added: "91"
- board text added: "92"
- board text added: "93"
- board text added: "94"
- board text added: "95"
- board text added: "96"
- board text added: "97"
- board text added: "98"
- board text added: "99"
- board text added: "A0"
- board text added: "A1"
- board text added: "A10"
- board text added: "A11"
- board text added: "A12"
- board text added: "A13"
- board text added: "A14"
- board text added: "A15"
- board text added: "A2"
- board text added: "A3"
- board text added: "A4"
- board text added: "A5"
- board text added: "A6"
- board text added: "A7"
- board text added: "A8"
- board text added: "A9"
- board text added: "CLOCK"
- board text added: "Copyright © 2026 John Winans https://github.com/johnwinans/2070-S-100-bus-analyzer"
- board text added: "D01"
- board text added: "D02"
- board text added: "DI0"
- board text added: "DI1"
- board text added: "DI2"
- board text added: "DI3"
- board text added: "DI4"
- board text added: "DI5"
- board text added: "DI6"
- board text added: "DI7"
- board text added: "DO0"
- board text added: "DO3"
- board text added: "DO4"
- board text added: "DO5"
- board text added: "DO6"
- board text added: "DO7"
- board text added: "PICO RESET"
- board text added: "S-100"
- board text added: "S-100 Bus Waveform Analyzer"
- board text added: "TRIGGER"
- board text added: "USB-C POWER ONLY"
- board text added: "USBC5"
- board text added: "VSYS"
- board text added: "sHLTA"
- board text added: "sINP"
- board text added: "sINTA"
- board text added: "sM1"
- board text added: "sMEMR"
- board text added: "sOUT"
- board text added: "~{ERROR}"
- board text added: "~{PHANT}"
- board text added: "~{POC}"
- board text added: "~{pDBIN}"
- board text added: "~{pWR}"
- board text added: "~{sWO}"
- board text removed: "~{PHANTOM}"

Commit message: Acute angles
Routing:
- net Net-(A3-GPIO19): track 41.5 -> 51.2 mm
- net Net-(A5-GPIO2): track 73.4 -> 78.4 mm
- net Net-(A5-GPIO4): track 68.1 -> 73.0 mm
- net Net-(A5-GPIO3): track 70.8 -> 75.5 mm
- net Net-(A5-GPIO5): track 65.5 -> 69.8 mm
- net Net-(A5-GPIO6): track 60.3 -> 64.2 mm
- net Net-(A5-GPIO7): track 57.6 -> 61.5 mm
- net Net-(A2-GPIO2): track 85.4 -> 89.0 mm
- net Net-(A5-GPIO9): track 52.3 -> 55.7 mm
- net Net-(A5-GPIO8): track 55.0 -> 58.3 mm
- net Net-(A2-GPIO3): track 82.8 -> 85.9 mm
- net Net-(A1-GPIO4): track 78.5 -> 81.6 mm
- net Net-(A1-GPIO2): track 83.8 -> 86.8 mm
- net Net-(A5-GPIO10): track 54.6 -> 57.6 mm
- net Net-(A4-GPIO2): track 86.4 -> 89.3 mm
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