File: 2070-S-100-bus-analyzer.kicad_pcb (KiCad board)
At the start: 4 copper layers, 254 x 137.8 mm, 85 parts, among them J10 Conn_02x13_Odd_Even, J11 Conn_02x13_Odd_Even, J12 USB4105-GF-A, J13 Conn_01x01, J14 Conn_01x01, J15 Conn_01x02, J16 Conn_01x02, J17 Conn_01x02, J18 Conn_01x02, J19 Conn_01x02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

Commit message: DRC cleanup
Parts:
- turned J13 to 90 degrees
- turned J14 to 90 degrees
Routing:
- net Net-(A3-3V3): vias 4 -> 3
- net GND: vias 66 -> 67
